File: pcb/_autosave-Guepard.kicad_pcb (KiCad board)
At the start: 2 copper layers, 205 parts, among them J1 USB_B-micro, J5 TE-776163, K2 CONN_3, P2 CONN_1, P27 BDM, P3 CONN_1, P4 CONN_1, P5 CONN_1, P9 BATT1, Q1 MOS_N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

Commit message: MPX4250 footprint
Routing:
- net GROUND: track 339.3 -> 277.3 mm
- net /Communication/USB-GND: track 88.5 -> 68.6 mm
Changed lines of the file:
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@@
   (general
     (links 415)
-    (no_connects 3)
-    (area 196.269199 67.234999 381.083821 186.62)
+    (no_connects 8)
+    (area 196.269199 67.234999 381.083821 183.675)
     (thickness 1.6)
     (drawings 52)
-    (tracks 1292)
+    (tracks 1268)
     (zones 0)
     (modules 205)
@@
     (add_net EXTAL)
     (add_net Fuel-Pump-Drive)
+    (add_net GROUND)
     (add_net IAT)
     (add_net IAT-Sensor)
@@
     (uvia_drill 0.127)
     (add_net FP-Relay)
-    (add_net GROUND)
     (add_net Output-Ground)
     (add_net Spare-LSD-1)
@@
   (segment (start 358.648 140.462) (end 355.6 140.462) (width 0.35) (layer Dessus.Cu) (net 6))
   (segment (start 361.5055 140.462) (end 358.648 140.462) (width 0.35) (layer Dessus.Cu) (net 6))
-  (segment (start 358.648 143.002) (end 364.236 143.002) (width 0.35) (layer Dessus.Cu) (net 7) (status 400000))
-  (segment (start 366.74552 134.08152) (end 365.85398 134.08152) (width 0.35) (layer Dessus.Cu) (net 7) (status 800000))
-  (segment (start 367.284 134.62) (end 366.74552 134.08152) (width 0.35) (layer Dessus.Cu) (net 7))
-  (segment (start 367.284 137.668) (end 367.284 134.62) (width 0.35) (layer Dessus.Cu) (net 7))
-  (segment (start 367.03 137.922) (end 367.284 137.668) (width 0.35) (layer Dessus.Cu) (net 7))
-  (segment (start 367.03 140.208) (end 367.03 137.922) (width 0.35) (layer Dessus.Cu) (net 7))
-  (segment (start 364.236 143.002) (end 367.03 140.208) (width 0.35) (layer Dessus.Cu) (net 7))
-  (segment (start 355.6 143.002) (end 358.648 143.002) (width 0.35) (layer Dessus.Cu) (net 7) (status C00000))
   (segment (start 358.902 136.144) (end 358.902 136.652) (width 0.35) (layer Dessus.Cu) (net 7))
   (segment (start 348.67088 138.50112) (end 348.67088 139.74318) (width 0.35) (layer Dessus.Cu) (net 7))
@@
   (segment (start 302.6029 122.3391) (end 302.006 122.936) (width 0.35) (layer Dessus.Cu) (net 21))
   (segment (start 266.192 131.318) (end 266.192 133.858) (width 0.35) (layer Dessous.Cu) (net 21))
-  (segment (start 346.71 97.79) (end 349.504 97.79) (width 0.55) (layer Dessus.Cu) (net 22) (status 400000))
-  (segment (start 350.52 98.806) (end 350.52 110.998) (width 0.55) (layer Dessus.Cu) (net 22) (status 800000))
-  (segment (start 349.504 97.79) (end 350.52 98.806) (width 0.55) (layer Dessus.Cu) (net 22))
-  (segment (start 340.614 81.534) (end 340.36 81.534) (width 0.55) (layer Dessus.Cu) (net 22) (status C00000))
-  (segment (start 330.2 83.058) (end 320.294 83.058) (width 0.55) (layer Dessus.Cu) (net 22) (status 800000))
-  (segment (start 333.502 79.756) (end 330.2 83.058) (width 0.55) (layer Dessus.Cu) (net 22))
-  (segment (start 338.582 79.756) (end 333.502 79.756) (width 0.55) (layer Dessus.Cu) (net 22))
-  (segment (start 340.36 81.534) (end 338.582 79.756) (width 0.55) (layer Dessus.Cu) (net 22) (status 400000))
-  (segment (start 289.814 129.032) (end 289.306 129.032) (width 0.35) (layer Dessus.Cu) (net 22) (status C00000))
-  (segment (start 275.59 140.208) (end 273.05 140.208) (width 0.35) (layer Dessus.Cu) (net 22) (status 800000))
-  (segment (start 276.606 139.192) (end 275.59 140.208) (width 0.35) (layer Dessus.Cu) (net 22))
-  (segment (start 276.606 137.922) (end 276.606 139.192) (width 0.35) (layer Dessus.Cu) (net 22))
-  (segment (start 279.146 135.382) (end 276.606 137.922) (width 0.35) (layer Dessus.Cu) (net 22))
-  (segment (start 282.956 135.382) (end 279.146 135.382) (width 0.35) (layer Dessus.Cu) (net 22))
-  (segment (start 289.306 129.032) (end 282.956 135.382) (width 0.35) (layer Dessus.Cu) (net 22) (status 400000))
-  (segment (start 326.3265 82.6135) (end 326.3265 81.57972) (width 0.35) (layer Dessus.Cu) (net 22) (status 800000))
   (segment (start 344.10904 147.42414) (end 344.10904 157.41904) (width 0.35) (layer Dessus.Cu) (net 22))
   (segment (start 362.10748 158.90748) (end 362.10748 160.42386) (width 0.35) (layer Dessus.Cu) (net 22))
