File: pcb/Digital-Inputs.sch (KiCad schematic (older format))
At the start: 20 parts, among them U10 74V1T04STR

Commit message: schematics update
Parts:
- removed D35: +12VBRVLED, symbol LED
- removed D97, D99: 1N5818-TP, symbol DIODESCH
- removed D98: 4.7V, symbol ZENER
- removed R59, R60, R61: 1k, symbol R
- removed R62, R64: 2k4, symbol R
- removed U10: 74V1T04STR, symbol 74V1T04STR
- added P4, P5: CONN_1, symbol CONN_1
Connections:
- net labels added: 5vdc
- net labels removed: 5vdc-analog, 5vdc-cpu, BRV-12v, PE0, PE1, PJ0, PJ1
- wire segments 46 -> 22
- no-connect marks 2 -> 0
Other:
- note added: "Connect P4 to P2 for Spare Digital 1\nConnect P5 to P3 for Spare Digital 2"
- note removed: "Wake Up Signal Conditioning"
