File: pcb/Outputs.sch (KiCad schematic (older format))
At the start: 60 parts, among them K1 CONN_3, Q10 VNN7NV0413TR, Q11 VNN7NV0413TR, Q5 VNN7NV0413TR, Q6 VNN7NV0413TR, Q9 VNN7NV0413TR, U12 TC442XA, U14 NC7WZ86K8X, U15 NC7WZ86K8X, U9 TC442XA

Commit message: replace TC442xa with TC4427
Parts:
- U12, U9: value TC442XA -> TC4427AVOA
Changed lines of the file:
@@
-EESchema Schematic File Version 2  date 23/05/2013 15:10:10
+EESchema Schematic File Version 2  date 24/05/2013 14:40:27
 LIBS:opto
 LIBS:power
@@
 Sheet 6 8
 Title "Guepard PCB for FreeEMS"
-Date "23 may 2013"
+Date "24 may 2013"
 Rev "0.1-alpha"
 Comp ""
@@
 12vdc-switched-outputs
 $Comp
-L GND #PWR034
+L GND #PWR42
 U 1 1 51778FC4
 P 6300 6250
-F 0 "#PWR034" H 6300 6250 30  0001 C CNN
+F 0 "#PWR42" H 6300 6250 30  0001 C CNN
 F 1 "GND" H 6300 6180 30  0001 C CNN
 	1    6300 6250
@@
 Output-Ground
 $Comp
-L GND #PWR035
+L GND #PWR37
 U 1 1 51778FB5
 P 2300 7250
-F 0 "#PWR035" H 2300 7250 30  0001 C CNN
+F 0 "#PWR37" H 2300 7250 30  0001 C CNN
 F 1 "GND" H 2300 7180 30  0001 C CNN
 	1    2300 7250
@@
 $EndComp
 $Comp
-L GND #PWR036
+L GND #PWR39
 U 1 1 51768E45
 P 5150 4100
-F 0 "#PWR036" H 5150 4100 30  0001 C CNN
+F 0 "#PWR39" H 5150 4100 30  0001 C CNN
 F 1 "GND" H 5150 4030 30  0001 C CNN
 	1    5150 4100
@@
 $EndComp
 $Comp
-L GND #PWR037
+L GND #PWR44
 U 1 1 51768E41
 P 7100 2950
-F 0 "#PWR037" H 7100 2950 30  0001 C CNN
+F 0 "#PWR44" H 7100 2950 30  0001 C CNN
 F 1 "GND" H 7100 2880 30  0001 C CNN
 	1    7100 2950
@@
 $EndComp
 $Comp
-L GND #PWR038
+L GND #PWR41
 U 1 1 51768E40
 P 5950 3650
-F 0 "#PWR038" H 5950 3650 30  0001 C CNN
+F 0 "#PWR41" H 5950 3650 30  0001 C CNN
 F 1 "GND" H 5950 3580 30  0001 C CNN
 	1    5950 3650
@@
 $EndComp
 $Comp
-L GND #PWR039
+L GND #PWR40
 U 1 1 51768DDF
 P 5950 2150
-F 0 "#PWR039" H 5950 2150 30  0001 C CNN
+F 0 "#PWR40" H 5950 2150 30  0001 C CNN
 F 1 "GND" H 5950 2080 30  0001 C CNN
 	1    5950 2150
@@
 $EndComp
 $Comp
-L GND #PWR040
+L GND #PWR43
 U 1 1 51768D8C
 P 6950 1250
-F 0 "#PWR040" H 6950 1250 30  0001 C CNN
+F 0 "#PWR43" H 6950 1250 30  0001 C CNN
 F 1 "GND" H 6950 1180 30  0001 C CNN
 	1    6950 1250
@@
 $EndComp
 $Comp
-L GND #PWR041
+L GND #PWR50
 U 1 1 517689CF
 P 10650 4000
-F 0 "#PWR041" H 10650 4000 30  0001 C CNN
+F 0 "#PWR50" H 10650 4000 30  0001 C CNN
 F 1 "GND" H 10650 3930 30  0001 C CNN
 	1    10650 4000
@@
 Ignitor3
 $Comp
-L GND #PWR042
+L GND #PWR49
 U 1 1 5176873D
 P 10650 2500
-F 0 "#PWR042" H 10650 2500 30  0001 C CNN
+F 0 "#PWR49" H 10650 2500 30  0001 C CNN
 F 1 "GND" H 10650 2430 30  0001 C CNN
 	1    10650 2500
@@
 AR Path="/4F0D82A1/509C864F" Ref="U12"  Part="1"
 F 0 "U12" H 8385 3691 60  0000 C CNN
-F 1 "TC442XA" H 8403 3121 60  0000 C CNN
+F 1 "TC4427AVOA" H 8403 3121 60  0000 C CNN
 	1    8400 3400
 	1    0    0    -1
@@
 $EndComp
 $Comp
-L GND #PWR043
+L GND #PWR45
 U 1 1 509C8646
 P 7650 3450
-F 0 "#PWR043" H 7650 3450 30  0001 C CNN
+F 0 "#PWR45" H 7650 3450 30  0001 C CNN
 F 1 "GND" H 7650 3380 30  0001 C CNN
 	1    7650 3450
@@
 NoConn ~ 7850 3250
 $Comp
-L GND #PWR044
+L GND #PWR48
 U 1 1 509C8641
 P 9750 2900
-F 0 "#PWR044" H 9750 2900 30  0001 C CNN
+F 0 "#PWR48" H 9750 2900 30  0001 C CNN
 F 1 "GND" H 9750 2830 30  0001 C CNN
 	1    9750 2900
@@
 JP11 selects either\n5v or 12v \nDriver IC Supply
 $Comp
-L GND #PWR045
+L GND #PWR47
 U 1 1 5092C12A
 P 9700 1650
-F 0 "#PWR045" H 9700 1650 30  0001 C CNN
+F 0 "#PWR47" H 9700 1650 30  0001 C CNN
 F 1 "GND" H 9700 1580 30  0001 C CNN
 	1    9700 1650
@@
 $EndComp
 $Comp
-L GND #PWR046
+L GND #PWR46
 U 1 1 5092BF20
 P 7700 1950
-F 0 "#PWR046" H 7700 1950 30  0001 C CNN
+F 0 "#PWR46" H 7700 1950 30  0001 C CNN
 F 1 "GND" H 7700 1880 30  0001 C CNN
 	1    7700 1950
@@
 $EndComp
 $Comp
-L GND #PWR047
+L GND #PWR38
 U 1 1 5092BF09
 P 5150 2600
-F 0 "#PWR047" H 5150 2600 30  0001 C CNN
+F 0 "#PWR38" H 5150 2600 30  0001 C CNN
 F 1 "GND" H 5150 2530 30  0001 C CNN
 	1    5150 2600
@@
 P 8400 1900
 F 0 "U9" H 8385 2191 60  0000 C CNN
-F 1 "TC442XA" H 8403 1621 60  0000 C CNN
+F 1 "TC4427AVOA" H 8403 1621 60  0000 C CNN
 	1    8400 1900
 	1    0    0    -1
@@
 12vdc-switched-outputs
 $Comp
-L GND #PWR048
+L GND #PWR36
 U 1 1 4F2F3E3F
 P 2300 5450
-F 0 "#PWR048" H 2300 5450 30  0001 C CNN
+F 0 "#PWR36" H 2300 5450 30  0001 C CNN
 F 1 "GND" H 2300 5380 30  0001 C CNN
 	1    2300 5450
@@
 $EndComp
 $Comp
-L GND #PWR049
+L GND #PWR35
 U 1 1 4F2F3E2D
 P 2300 3650
-F 0 "#PWR049" H 2300 3650 30  0001 C CNN
+F 0 "#PWR35" H 2300 3650 30  0001 C CNN
 F 1 "GND" H 2300 3580 30  0001 C CNN
 	1    2300 3650
@@
 $EndComp
 $Comp
-L GND #PWR050
+L GND #PWR34
 U 1 1 4F2F3E0C
 P 2300 1850
-F 0 "#PWR050" H 2300 1850 30  0001 C CNN
+F 0 "#PWR34" H 2300 1850 30  0001 C CNN
 F 1 "GND" H 2300 1780 30  0001 C CNN
 	1    2300 1850

Commit message: schematics update
Parts:
- removed C12, C14: 0.1uF, symbol C
- removed D52, D54: LED, symbol LED
- removed D53, D55: 1N4148, symbol DIODE
- removed K1: CONN_3, symbol CONN_3
- removed Q5, Q6: VNN7NV0413TR, symbol MOSFET_N
- removed R69, R78: 2.4k, symbol R
- removed R7, R71: 1k, symbol R
- removed R70, R79: 100k, symbol R
- removed U14, U15: NC7WZ86K8X, symbol NC7WZ86K8X
- R100, R101, R91, R92: value 150 -> 160
Connections:
- net labels added: 5vdc
- net labels removed: 5vdc-analog, PP6, PP7, Spare-LSD-3, Spare-LSD-4
- wire segments 127 -> 80
Other:
- note removed: "Jumper to select either\n5V or GND for XOR Input"
- note removed: "Low Side Driver #3 Output"
- note removed: "Low Side Driver #4 Output"
- moved on the sheet: R102, R103, R104, R105, R87, R88, R89, R90
