File: pcb/Guepard.kicad_pcb (KiCad board)
At the start: 2 copper layers, 205 parts, among them J1 USB_B-micro, J5 TE-776163, K2 CONN_3, P2 CONN_1, P27 BDM, P3 CONN_1, P4 CONN_1, P5 CONN_1, P9 BATT1, Q1 MOS_N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

Commit message: Ground plane under MCU - RPM traces - power capacitor for MCU
The ground plane under the Freescale MCU should look like the suggested
PCB design in the Freescale 9S12XDP512 datasheet
Parts:
- P9: footprint keystone_103 -> PIN_ARRAY_2
- U5: value M41T56M6 -> DS1307ZN+
- U7: footprint msoic-8 -> dil_8-300
- moved P9 23.4 mm to (334.0, 99.6), turned to 270 degrees
- moved R12 11.4 mm to (347.5, 126.7), turned to 180 degrees
- moved U7 5.18 mm to (348.2, 118.9)
- moved C25 3.59 mm to (348.2, 111.5), turned to 180 degrees
Routing:
- net 5vdc: track 630.6 -> 664.7 mm
- net GROUND: track 339.3 -> 362.1 mm
- net N-00000101: track 23.3 -> 8.17 mm
- net CPU-TXCAN0: track 34.5 -> 47.2 mm
- net RPM-Crank-IN+: track 309.2 -> 304.0 mm
- net N-00000260: track 2.08 -> 6.18 mm
- net N-00000255: track 26.6 -> 22.7 mm
- net COOLANT: track 29.4 -> 32.9 mm
- net CPU-RXCAN0: track 34.0 -> 36.0 mm, vias 2 -> 0
- net N-00000261: track 22.0 -> 21.0 mm
